Commit message: Updated URDF

File: Hardware/Mini/urdf_out/bb_mini/urdf/bb_mini.urdf (robot description, URDF)
Before this commit: robot bb_mini, 3 links, 2 joints
Links:
- link base_link: mass 0.099831 -> 0.192203558749535
- link left_wheel: mass 0.0043782 -> 0.00496078957070453
- link right_wheel: mass 0.0043782 -> 0.00496078957070453
